File: extras/PCB/Phoenix_shield_v0.1/Phoenix_FC_shield.brd (EAGLE design)
At the start: 50 x 50 mm, 51 parts, among them T1 BC817-40SMD, T2 BC817-40SMD

Commit message: PCB - tiny resistor value changes
Parts:
- R14: value 2K -> 1k8
Changed lines of the file:
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@@
 <attribute name="NAME" x="31.238" y="4.816" size="0.8128" layer="25"/>
 </element>
-<element name="R14" library="resistor" package="R0805" value="2K" x="29.1" y="2.3" smashed="yes">
+<element name="R14" library="resistor" package="R0805" value="1k8" x="29.1" y="2.3" smashed="yes">
 <attribute name="NAME" x="31.238" y="0.516" size="0.8128" layer="25"/>
 </element>
